File: tlcr-raspberry.sch (EAGLE design)
At the start: 103 parts, among them IC1 BUCK_REGULATOR_SIC413

Commit message: Schematic seems to be ready.
Parts:
- removed 0.C5, 10.C2, 12.C10, 12.C11, 12.C12, 12.C3, 12.C4, 12.C8, 6.C0, 9.C0, 9.C1: 100nF, RC_and_L:C-EUC0805
- removed 0.MCU1: AT32UCL016/32/64_TQFP48, tlcamera_rail_to_manufacture:AT32UCL016/32/64_TQFP48
- removed 1.ENC1, 1.ENC2, 1.ENC3: ENCODER_QUADRATE_WITH_BUTTON_ENCODER_PEC11-4XXXF-SXXXX, tlcamera_rail_to_manufacture:ENCODER_QUADRATE_WITH_BUTTON_ENCODER_PEC11-4XXXF-SXXXX
- removed 1.SW_LM_1, 1.SW_LM_2: CONNECTOR_2PIN, connectors:CONNECTOR_2PIN1X2_WIRE
- removed 10.C0, 10.C1, 12.C1, 12.C2, 12.C5, 12.C6, 7.C1, 7.C2: 22uF, RC_and_L:CPOL-EUE1.5-5
- removed 10.IC0: TCM828_VOLTAGE_INVERTER, tlcamera_rail_to_manufacture:TCM828_VOLTAGE_INVERTER
- removed 10.LCD0: LCD_WITH_COMMON_INTERFACE_FDCC0802C-NSWBBH-91LE, tlcamera_rail_to_manufacture:LCD_WITH_COMMON_INTERFACE_FDCC0802C-NSWBBH-91LE
- removed 10.R0: 1k, tlcamera_rail_to_manufacture:R-TRIMMER
- removed 11.CON0: 2.5MM-JACK-STEREO-CONNECTOR, tlcamera_rail_to_manufacture:2.5MM-JACK-STEREO-CONNECTOR
- removed 11.IC0, 11.IC1: HCPL-817, tlcamera_rail_to_manufacture:HCPL-817
- removed 11.R0, 11.R1: 500, RC_and_L:R-EU_R0805
- removed 12.C0, 12.C7, 4.C1, 7.C0, 7.C3: 220uF, RC_and_L:CPOL-EUE3.5-8
- removed 12.C9: 4.7uF, RC_and_L:CPOL-EUE1.5-5
- removed 12.J0, 12.J1: CONNECTOR_1PINGND_PIN, connectors:CONNECTOR_1PINGND_PIN
- removed 12.L1: 15uH, tlcamera_rail_to_manufacture:LMCBFS7330-150MU
- removed 12.R1: 75k, RC_and_L:R-EU_R0805
- removed 12.R2, 4.R2, 4.R3, 5.R2, 5.R3, 9.R2, 9.R5: 10k, RC_and_L:R-EU_R0805
- removed 2.CON0, 3.CON0, 4.CON0, 5.CON0: CONNECTOR_2PIN1X2_MOTOR_COIL, connectors:CONNECTOR_2PIN1X2_MOTOR_COIL
- removed 2.IC0, 2.IC1, 3.IC0, 3.IC1, 4.IC0, 4.IC1, 5.IC0, 5.IC1: N_MOSFET_TSM2N7002, tlcamera_rail_to_manufacture:N_MOSFET_TSM2N7002
- removed 2.IC2, 2.IC3, 3.IC2, 3.IC3, 4.IC2, 4.IC3, 5.IC2, 5.IC3: P_MOSFET_NX2301P, tlcamera_rail_to_manufacture:P_MOSFET_NX2301P
- removed 2.IC4, 2.IC5, 3.IC4, 3.IC5, 4.IC4, 4.IC5, 5.IC4, 5.IC5: N_MOSFET_PMV16UN, tlcamera_rail_to_manufacture:N_MOSFET_PMV16UN
- removed 2.R0, 3.R0, 4.R0, 4.R1, 5.R0, 5.R1: 1k, RC_and_L:R-EU_R0805
- removed 6.IC0: FLASH_AT25DF021_SO8, tlcamera_rail_to_manufacture:FLASH_AT25DF021_SO8
- removed 7.CON7: MJ-180PH, tlcamera_rail_to_manufacture:MJ-180PH
- removed 7.IC0: REGULATOR_AP1117E33G-13, tlcamera_rail_to_manufacture:REGULATOR_AP1117E33G-13
- removed 9.CON0: USB-BWUERTH-ELECTRONIC-USB-B, tlcamera_rail_to_manufacture:USB-BWUERTH-ELECTRONIC-USB-B
- removed 9.IC0: FT232RL, tlcamera_rail_to_manufacture:FT232RL
- removed 9.R1: 4k7, RC_and_L:R-EU_R0805
- removed 9.R6: 1M, RC_and_L:R-EU_R0805
- added 0.C0: 22uF, RC_and_L:CPOL-EUE1.5-5
- added 0.C1, 1.C0, 1.C1, 1.C2, 1.C4, 2.C10, 2.C11, 2.C2, 2.C3, 3.C6, 3.C7: 100nF, RC_and_L:C-EUC0805
- added 1.ISPC: CONNECTOR_6PIN2X3_ISP, connectors:CONNECTOR_6PIN2X3_ISP
- added 1.MCU1: ATMEGA48-20PU-32TQFPTQFP32, ic:ATMEGA48-20PU-32TQFPTQFP32
- added 2.C0, 3.C4, 3.C5, 4.C8, 4.C9, 5.C3: 220nF, RC_and_L:C-EUC0805
- added 2.DRIVER, 3.DRIVER, 4.DRIVER: A4985, ic:A4985
- added 2.MCON, 3.MCON, 4.MCON: CONNECTOR_4PIN, connectors:CONNECTOR_4PIN
- added 2.TB1, 2.TB7, 2.TC2, 2.TC3, 2.TC4, 2.TC5, 2.TC6, 2.TD7, 5.+24V, 5.+5V, 5.GND: CONNECTOR_1PIN1X1_HEADER, connectors:CONNECTOR_1PIN1X1_HEADER
- added 3.C1, 3.C2, 3.C3: (no value), RC_and_L:C-EUC0805
- added 3.R4, 3.R5, 4.R7, 4.R8: (no value), RC_and_L:R-EU_R2010
- added 3.R6, 4.R9: (no value), RC_and_L:R-EU_R0805
- added 5.C1: 22uF, RC_and_L:CPOL-EU140CLH-0810
- added 5.C2: 220uF, RC_and_L:CPOL-EU140CLH-0810
- added 5.PWRCON: CONNECTOR_2PIN1X2_WIRE, connectors:CONNECTOR_2PIN1X2_WIRE
- 0.CON1: value CONNECTOR_3PINAWIRE -> USB-BWUERTH-ELECTRONIC-USB-B; device connectors:CONNECTOR_3PINAWIRE -> connectors:USB-BWUERTH-ELECTRONIC-USB-B
- 2.C1: value 220uF -> 220nF; device RC_and_L:CPOL-EUE3.5-8 -> RC_and_L:C-EUC0805
- 2.R1: value 1k -> (none); device RC_and_L:R-EU_R0805 -> RC_and_L:R-EU_R2010
- 2.R2: value 10k -> (none); device RC_and_L:R-EU_R0805 -> RC_and_L:R-EU_R2010
- 2.R3, 3.R2, 3.R3: value 10k -> (none)
- 3.R1: value 1k -> (none)
- IC1: value BUCK_REGULATOR_SIC413 -> FT232RL; device tlcamera_rail_to_manufacture:BUCK_REGULATOR_SIC413 -> ic:FT232RL
Connections:
- removed net #RESET(AWIRE_DATA): 0.CON1.P$3, 0.MCU1.RESET_N(AWIRE_DATA)
- removed net +12V: 12.C0.+, 12.C1.+, 12.C2.+, 12.C3.1, 7.C0.+, 7.C1.+, 7.CON7.V+, 7.IC0.VIN, IC1.V_IN
- removed net +3V3: 0.C2.1, 0.C3.1, 0.CON1.P$1, 0.MCU1.VDDIN, 0.MCU1.VDDIO, 0.MCU1.VDDIO@1, 10.C2.1, 10.IC0.VIN, 10.LCD0.LED+, 10.LCD0.VDD, 6.C0.1, 6.IC0.VCC, 7.C2.+, 7.C3.+, 7.IC0.VOUT, 7.IC0.VOUT@1, 9.C0.1, 9.IC0.VCC, 9.IC0.VCCIO
- removed net MOTOR_VCC: 12.C4.1, 12.C5.+, 12.C6.+, 12.C7.+, 12.C8.1, 12.L1.2, 12.R1.2, 2.C1.+, 2.IC2.S, 2.IC3.S, 2.R0.2, 2.R1.2, 3.IC2.S, 3.IC3.S, 3.R0.2, 3.R1.2, 4.C1.+, 4.IC2.S, 4.IC3.S, 4.R0.2, 4.R1.2, 5.IC2.S, 5.IC3.S, 5.R0.2, 5.R1.2
- removed net PA00(TXD0): 0.MCU1.PA00(TXD0/NPCS2/PWMA0), 9.IC0.RXD
- removed net PA01(RXD0): 0.MCU1.PA01(RXD0/NPCS3/PWMA1), 9.IC0.TXD
- removed net PA02(RTS0): 0.MCU1.PA02(RTS0/PWMA2), 9.IC0.CTS#
- removed net PA03(CTS0): 0.MCU1.PA03(NPCS1/PWMA3), 9.IC0.RTS#
- removed net PA04(MISO): 0.MCU1.PA04(MISO/PWMA4), 6.IC0.SO
- removed net PA05(MOSI): 0.MCU1.PA05(MOSI/PWMA5), 6.IC0.SI
- removed net PA06(SCK): 0.MCU1.PA06(SCK/PWMA6), 6.IC0.SCK
- removed net PA07(NPCS0): 0.MCU1.PA07(NPCS0/EXINT0/PWMA7), 6.IC0.#CS
- removed net PA08: 0.MCU1.PA08(NPCS2/PWMA8), 10.LCD0.LED-
- removed net PA09: 0.MCU1.PA09(NPCS3/PWMA9/EXTINT1), 1.ENC1_QUADR.A
- removed net PA10: 0.MCU1.PA10(PWMA10), 1.ENC1_QUADR.B
- removed net PA11: 0.MCU1.PA11(PWMA11), 1.ENC2_QUADR.B
- removed net PA12: 0.MCU1.PA12(PWMA12), 1.ENC3_SW.P$1, 1.SW_LM_1.P$1
- removed net PA13: 0.MCU1.PA13(PWMA13/EXTINT2), 1.ENC2_QUADR.A
- removed net PA14: 0.MCU1.PA14(PWMA14), 1.ENC2_SW.P$1, 1.SW_LM_2.P$1
- removed net PA15: 0.MCU1.PA15(PWMA15), 1.ENC3_QUADR.A
- removed net PA16: 0.MCU1.PA16(PWMA17), 1.ENC1_SW.P$2, 1.ENC2_SW.P$2, 1.ENC3_SW.P$2
- removed net PA17: 0.MCU1.PA17(PWMA17), 10.LCD0.RS
- removed net PA18: 0.MCU1.PA18(PWMA18), 10.LCD0.E
- removed net PA19: 0.MCU1.PA19(PWMA19), 11.R1.2
- removed net PA20: 0.MCU1.PA20(PWMA20), 10.LCD0.DB4
- removed net PA21: 0.MCU1.PA21(PWMA21), 10.LCD0.DB5
- removed net PA22: 0.MCU1.PA22(CTS0/PWMA22), 10.LCD0.DB6
- removed net PB00: 0.MCU1.PB00(NPCS0/PWMA23), 10.LCD0.DB7
- removed net PB01: 0.MCU1.PB01(SCK/PWMA24), 4.IC0.G, 4.IC5.G, 4.R3.2
- removed net PB02: 0.MCU1.PB02(MISO/PWMA25), 4.IC1.G, 4.IC4.G, 4.R2.2
- removed net PB03: 0.MCU1.PB03(MOSI/PWMA26), 5.IC0.G, 5.IC5.G, 5.R3.2
- removed net PB04: 0.MCU1.PB04(PWMA27), 5.IC1.G, 5.IC4.G, 5.R2.2
- removed net PB05: 0.MCU1.PB05(PWMA28), 2.IC0.G, 2.IC5.G, 2.R3.2
- removed net PB06: 0.MCU1.PB06(EXTINT0/PWMA29), 2.IC1.G, 2.IC4.G, 2.R2.2
- removed net PB07: 0.MCU1.PB07(EINT1/EXTINT1/PWMA30), 3.IC0.G, 3.IC5.G, 3.R3.2
- removed net PB08: 0.MCU1.PB08(EXTINT2/PWMA31), 3.IC1.G, 3.IC4.G, 3.R2.2
- removed net PB09: 0.MCU1.PB09(EXTINT3/PWMA32), 1.ENC3_QUADR.B
- removed net PB10: 0.MCU1.PB10(EXTINT4/PWMA33), 11.R0.2
- removed net PB11: 0.MCU1.PB11(EXTINT5/PWMA34), 1.SW_LM_1.P$2, 1.SW_LM_2.P$2
- removed net PB12: 0.MCU1.PB12(PWMA35), 1.ENC1_SW.P$1
- new net !RESET: 1.ISPC.P$4, 1.MCU1.PC6(!RESET)
- new net +24V: 2.C11.2, 2.C3.2, 2.DRIVER.VBB1, 2.DRIVER.VBB2, 3.C7.2, 3.DRIVER.VBB1, 3.DRIVER.VBB2, 4.DRIVER.VBB1, 4.DRIVER.VBB2, 5.+24V.P$1, 5.C1.+, 5.C2.+, 5.C3.1, 5.PWRCON.P$1
- new net +5V: 0.C0.+, 0.C1.1, 0.C2.1, 0.C3.1, 0.CON1.VCC@1, 1.C0.1, 1.C1.1, 1.C2.1, 1.ISPC.P$1, 1.MCU1.AVCC, 1.MCU1.VCC@1, 1.MCU1.VCC@2, 2.C0.1, 2.DRIVER.VDD, 3.C4.1, 3.DRIVER.VDD, 4.C8.1, 4.DRIVER.VDD, 5.+5V.P$1, IC1.VCC, IC1.VCCIO
- new net ADC6: 1.MCU1.ADC6
- new net ADC7: 1.MCU1.ADC7
- new net B0: 1.MCU1.PB0, 3.DRIVER.STEP
- new net B1: 1.MCU1.PB1, 2.TB1.P$1, 3.R3.2
- new net B2: 1.MCU1.PB2, 3.R1.2
- new net B6: 1.MCU1.PB6, 3.DRIVER.DIR
- new net B7: 1.MCU1.PB7, 2.DRIVER.!ENABLE, 2.TB7.P$1, 3.DRIVER.!ENABLE, 4.DRIVER.!ENABLE
- new net C0: 1.MCU1.PC0(ADC0), 4.DRIVER.STEP
- new net C1: 1.MCU1.PC1(ADC1), 4.DRIVER.DIR
- new net C2: 1.MCU1.PC2(ADC2), 2.DRIVER.STEP, 2.TC2.P$1
- new net C3: 1.MCU1.PC3(ADC3), 2.DRIVER.DIR, 2.TC3.P$1
- new net C4: 1.MCU1.PC4(ADC4), 2.DRIVER.MS1, 2.TC4.P$1, 3.DRIVER.MS1, 4.DRIVER.MS1
- new net C5: 1.MCU1.PC5(ADC5), 2.DRIVER.MS2, 2.TC5.P$1, 3.DRIVER.MS2, 4.DRIVER.MS2
- new net D2: 1.MCU1.PD2(INT0)
- new net D3: 1.MCU1.PD3(INT1), 3.R2.2
- new net D4: 1.MCU1.PD4
- new net D5: 1.MCU1.PD5(OC0B)
- new net D6: 1.MCU1.PD6(OC0A), 2.DRIVER.!SLEEP, 2.TC6.P$1, 3.DRIVER.!SLEEP, 4.DRIVER.!SLEEP
- new net D7: 1.MCU1.PD7(AIN1), 2.DRIVER.!RESET, 2.TD7.P$1, 3.DRIVER.!RESET, 4.DRIVER.!RESET
- new net MISO: 1.ISPC.P$2, 1.MCU1.PB4(MISO)
- new net MOSI: 1.ISPC.P$3, 1.MCU1.PB3(MOSI)
- new net N$39: 4.R7.1
- new net N$40: 4.DRIVER.ROSC, 4.R9.2
- new net N$41: 3.C1.1, 3.DRIVER.REF, 3.R1.1
- new net N$43: 3.C2.1, 3.R2.1, 4.DRIVER.REF
- new net N$45: 2.DRIVER.REF, 3.C3.1, 3.R3.1
- new net N$46: 3.C3.2
- new net RXD: 1.MCU1.PD0(RXD), IC1.TXD
- new net SCK: 1.ISPC.P$5, 1.MCU1.PB5(SCK)
- new net TXD: 1.MCU1.PD1(TXD), IC1.RXD
- net GND: now also 0.C0.-, 0.C1.2, 0.CON1.GND, 0.CON1.SHIELD@1, 0.CON1.SHIELD@2, 1.C0.2, 1.C1.2, 1.C2.2, 1.C4.2, 1.ISPC.P$6, 1.MCU1.GND@1, 1.MCU1.GND@2, 1.MCU1.GND@3, 2.C0.2, 2.C1.2, 2.DRIVER.GND, 2.DRIVER.GND@1, 3.C1.2, 3.C2.2, 3.C4.2, 3.C5.2, 3.DRIVER.GND, 3.DRIVER.GND@1, 3.R5.1, 3.R6.1, 4.C8.2, 4.C9.2, 4.DRIVER.GND, 4.DRIVER.GND@1, 4.R8.1, 4.R9.1, 5.C1.-, 5.C2.-, 5.C3.2, 5.GND.P$1, 5.PWRCON.P$2, IC1.AGND, IC1.GND@0, IC1.GND@1, IC1.GND@2, IC1.TEST; no longer 0.C5.2, 0.CON1.P$2, 0.MCU1.GND, 0.MCU1.GND@1, 0.MCU1.GND@2, 0.MCU1.GND@3, 0.MCU1.GNDANA, 1.ENC1_QUADR.COM, 1.ENC1_QUADR.SHIELD, 1.ENC1_QUADR.SHIELD@1, 1.ENC2_QUADR.COM, 1.ENC2_QUADR.SHIELD, 1.ENC2_QUADR.SHIELD@1, 1.ENC3_QUADR.COM, 1.ENC3_QUADR.SHIELD, 1.ENC3_QUADR.SHIELD@1, 10.C0.+, 10.C2.2, 10.IC0.GND, 10.LCD0.RW, 10.LCD0.VSS, 10.R0.3, 11.IC0.CATHODE, 11.IC1.CATHODE, 12.C0.-, 12.C1.-, 12.C11.2, 12.C12.2, 12.C2.-, 12.C3.2, 12.C4.2, 12.C5.-, 12.C6.-, 12.C7.-, 12.C9.-, 12.J0.P$1, 12.J1.P$1, 12.R2.1, 2.C1.-, 2.IC0.S, 2.IC1.S, 2.IC4.S, 2.IC5.S, 3.IC0.S, 3.IC1.S, 3.IC4.S, 3.IC5.S, 3.R2.1, 3.R3.1, 4.C1.-, 4.IC0.S, 4.IC1.S, 4.IC4.S, 4.IC5.S, 4.R2.1, 4.R3.1, 5.IC0.S, 5.IC1.S, 5.IC4.S, 5.IC5.S, 5.R2.1, 5.R3.1, 6.C0.2, 6.IC0.GND, 7.C0.-, 7.C1.-, 7.C2.-, 7.C3.-, 7.CON7.GND, 7.IC0.GND, 9.C0.2, 9.C1.2, 9.CON0.GND, 9.CON0.SHIELD@1, 9.CON0.SHIELD@2, 9.IC0.AGND, 9.IC0.GND@0, 9.IC0.GND@1, 9.IC0.GND@2, 9.IC0.TEST, 9.R2.1, 9.R6.1, IC1.GND
- net N$1: now also 1.C4.1, 1.MCU1.AREF; no longer 9.C1.1, 9.IC0.3V3OUT
- net N$10: now also 2.DRIVER.OUT1A, 2.MCON.P$1; no longer 2.CON0.P$1, 2.IC2.D, 2.IC4.D
- net N$11: now also 2.DRIVER.OUT2A, 2.MCON.P$2; no longer 3.IC1.D, 3.IC3.G, 3.R1.1
- net N$12: now also 2.DRIVER.OUT1B, 2.MCON.P$3; no longer 3.CON0.P$2, 3.IC3.D, 3.IC5.D
- net N$13: now also 2.DRIVER.OUT2B, 2.MCON.P$4; no longer 10.LCD0.VO_CONTRAST, 10.R0.2
- net N$14: now also 2.DRIVER.SENSE1, 2.R1.2; no longer 3.CON0.P$1, 3.IC2.D, 3.IC4.D
- net N$15: now also 2.DRIVER.SENSE2, 2.R2.2; no longer 11.CON0.3, 11.CON0.4, 11.IC0.EMITTER, 11.IC1.EMITTER
- net N$16: now also 3.C6.1, 3.DRIVER.CP1; no longer 10.C1.+, 10.IC0.C+
- net N$17: now also 2.R1.1; no longer 10.C1.-, 10.IC0.C-
- net N$18: now also 3.C6.2, 3.DRIVER.CP2; no longer 4.IC0.D, 4.IC2.G, 4.R0.1
- net N$19: now also 2.DRIVER.ROSC, 2.R3.2; no longer 4.IC1.D, 4.IC3.G, 4.R1.1
- net N$2: now also 2.C1.1, 2.DRIVER.VREG; no longer 2.IC0.D, 2.IC2.G, 2.R0.1
- net N$20: now also 3.C7.1, 3.DRIVER.VCP; no longer 4.CON0.P$2, 4.IC3.D, 4.IC5.D
- net N$21: now also 3.DRIVER.OUT1A, 3.MCON.P$1; no longer 4.CON0.P$1, 4.IC2.D, 4.IC4.D
- net N$22: now also 3.DRIVER.OUT2A, 3.MCON.P$2; no longer 12.C11.1, 9.R5.2, 9.R6.2, IC1.COMP
- net N$23: now also 3.DRIVER.OUT1B, 3.MCON.P$3; no longer 10.C0.-, 10.IC0.VOUT, 10.R0.1
- net N$24: now also 3.DRIVER.OUT2B, 3.MCON.P$4; no longer 5.IC0.D, 5.IC2.G, 5.R0.1
- net N$25: now also 3.DRIVER.SENSE1, 3.R4.2; no longer 5.IC1.D, 5.IC3.G, 5.R1.1
- net N$26: now also 3.DRIVER.SENSE2, 3.R5.2; no longer 5.CON0.P$2, 5.IC3.D, 5.IC5.D
- net N$27: now also 3.R4.1; no longer 5.CON0.P$1, 5.IC2.D, 5.IC4.D
- net N$28: now also 3.DRIVER.ROSC, 3.R6.2; no longer 0.C4.1, 0.MCU1.VDDCORE
- net N$29: now also 4.C9.1, 4.DRIVER.VREG; no longer 12.C10.1, IC1.BOOT
- net N$3: now also 0.CON1.D+, IC1.USBDP; no longer 9.CON0.D-, 9.IC0.USBDM
- net N$30: now also 2.C10.1, 4.DRIVER.CP1; no longer 12.C8.2, 12.R1.1, 12.R2.2, IC1.FB
- net N$31: now also 2.C10.2, 4.DRIVER.CP2; no longer 11.CON0.1, 11.IC0.COLLECTOR
- net N$32: now also 2.C11.1, 4.DRIVER.VCP; no longer 12.C10.2, 12.L1.1, IC1.V_SW
- net N$33: now also 4.DRIVER.OUT1A, 4.MCON.P$1; no longer 12.C12.1, 9.R5.1
- net N$34: now also 4.DRIVER.OUT2A, 4.MCON.P$2; no longer 11.CON0.2, 11.IC1.COLLECTOR
- net N$35: now also 4.DRIVER.OUT1B, 4.MCON.P$3; no longer 0.C5.1, 0.MCU1.VDDANA
- net N$36: now also 4.DRIVER.OUT2B, 4.MCON.P$4; no longer 12.C9.+, IC1.V_REG
- net N$37: now also 4.DRIVER.SENSE1, 4.R7.2; no longer 11.IC0.ANODE, 11.R0.1
- net N$38: now also 4.DRIVER.SENSE2, 4.R8.2; no longer 11.IC1.ANODE, 11.R1.1
- net N$4: now also 0.CON1.D-, IC1.USBDM; no longer 9.CON0.D+, 9.IC0.USBDP
- net N$5: now also 2.C2.1, 2.DRIVER.CP1; no longer 9.CON0.VCC@1, 9.R1.2
- net N$6: now also 2.C2.2, 2.DRIVER.CP2; no longer 9.IC0.#RESET, 9.R1.1, 9.R2.2
- net N$7: now also 0.C4.1, IC1.3V3OUT; no longer 3.IC0.D, 3.IC2.G, 3.R0.1
- net N$8: now also 2.C3.1, 2.DRIVER.VCP; no longer 2.IC1.D, 2.IC3.G, 2.R1.1
- net N$9: now also 3.C5.1, 3.DRIVER.VREG; no longer 2.CON0.P$2, 2.IC3.D, 2.IC5.D
Other:
- note added: "BYBASS FOR FT232RL"
- note added: "BYPASS for Atmega48"
- note added: "Device low level voltages come from USB port"
- note added: "Input VCC filtering"
- note added: "Program MCU connector"
- note added: "VCC"
- note added: "VCCIO"
- note added: "[0]"
- note added: "[1]"
- note added: "[2]"
- note added: "[3]"
- note added: "[4]"
- note added: "[5]"
- note removed: "-3.3V"
- note removed: "3.3V POWER"
- note removed: "3.3V power for MCU and circuits."
- note removed: "BLUE"
- note removed: "Bypass"
- note removed: "Bypass condensator."
- note removed: "CAMERA TRIGGER"
- note removed: "Compensation"
- note removed: "Contrast adjust trimmer."
- note removed: "DC POWER CONNECTOR, INPUT (7-26V)"
- note removed: "Differential, place paraller, same length"
- note removed: "Display has internal current limiting resistor."
- note removed: "Encoder "knob" buttons."
- note removed: "Formula Vo=0.6V*(1+R1/R2)"
- note removed: "Forward current: (3.3V-1.2V) / Rs = XmA"
- note removed: "GND pin for oscilloscope"
- note removed: "H-Bridge, controls ROTATE axis stepper motor A coil."
- note removed: "H-Bridge, controls ROTATE axis stepper motor B coil."
- note removed: "H-Bridge, controls X axis stepper motor A coil."
- note removed: "H-Bridge, controls X axis stepper motor B coil."
- note removed: "LCD DISPLAY"
- note removed: "Limit SW buttons."
- note removed: "MCU"
- note removed: "MCU bypass condensators."
- note removed: "MEMORY, FLASH, IC"
- note removed: "MOTOR POWER, DC BUCK, OUTPUT ~6V, 4A MAX"
- note removed: "More memory is required for large text pages in terminal,"
- note removed: "PIC-COUNT Encoder."
- note removed: "PREFIX 0"
- note removed: "PREFIX 1"
- note removed: "PREFIX 10"
- note removed: "PREFIX 11"
- note removed: "PREFIX 12"
- note removed: "PREFIX 2"
- note removed: "PREFIX 3"
- note removed: "PREFIX 4"
- note removed: "PREFIX 5"
- note removed: "PREFIX 6"
- note removed: "PREFIX 7"
- note removed: "PREFIX 9"
- note removed: "Place near H-Bridge"
- note removed: "Prefix 13"
- note removed: "Programming connector, AWIRE"
- note removed: "R1+R2 should be 10-100k"
- note removed: "RED"
- note removed: "ROTATE MOTOR COIL A"
- note removed: "ROTATE MOTOR COIL B"
- note removed: "ROTATE-SPEED Encoder."
- note removed: "Removed"
- note removed: "Reset circuit is reguired, otherwise USB IC works unreliable."
- note removed: "TXD/RXD and CTS/RTS are crossed!"
- note removed: "Tested: Camera ground (3/4) to 1, Focus. To 2 take photo."
- note removed: "UI and LIMIT switches"
- note removed: "USB-UART CONVERTER IC"
- note removed: "Vref = 0.6V"
- note removed: "WHITE"
- note removed: "With this you can disable display BL"
- note removed: "X MOTOR COIL A"
- note removed: "X MOTOR COIL B"
- note removed: "X-SPEED Encoder."
- note removed: "YELLOW"
- note removed: "and later maybe for web pages over wlan API."
- moved on the sheet: 0.C2, 0.C3, 0.C4, 2.R1, 2.R2, 2.R3, 3.R1, 3.R2, 3.R3

Commit message: PCB layout ready.
Parts:
- removed 1.C2, 3.C6, 3.C7: 100nF, RC_and_L:C-EUC0805
- removed 2.C0: 220nF, RC_and_L:C-EUC0805
- removed 3.R5: (no value), RC_and_L:R-EU_R2010
- removed 3.R6: (no value), RC_and_L:R-EU_R0805
- added 2.C4, 2.C5: 100nF, RC_and_L:C-EUC0805
- added 2.R4: (no value), RC_and_L:R-EU_R2010
- added 4.C1: (no value), RC_and_L:C-EUC0805
- added 4.R1: (no value), RC_and_L:R-EU_R0805
- added 5.GND1: CONNECTOR_1PIN1X1_HEADER, connectors:CONNECTOR_1PIN1X1_HEADER
- 2.C1: value 220nF -> (none)
- 2.C2, 2.C3: value 100nF -> 220nF
- 2.R1, 2.R2: device RC_and_L:R-EU_R2010 -> RC_and_L:R-EU_R0805
- 2.R3, 3.R3: device RC_and_L:R-EU_R0805 -> RC_and_L:R-EU_R2010
- 3.C2, 3.C3: value (none) -> 220nF
- 3.C4, 3.C5: value 220nF -> 100nF
- renumbered 2.C10 to 4.C4, 2.C11 to 4.C5, 4.C8 to 4.C2, 4.C9 to 4.C3, 4.R7 to 4.R3, 4.R8 to 4.R4, 4.R9 to 4.R2
Connections:
- removed net N$17: 2.R1.1
- removed net N$27: 3.R4.1
- removed net N$39: 4.R3.1
- removed net N$46: 3.C3.2
- net +24V: now also 2.C5.2, 3.C5.2; no longer 2.C3.2, 3.C7.2
- net +5V: now also 2.C2.1, 3.C2.1; no longer 1.C2.1, 2.C0.1, 3.C4.1
- net B1: now also 2.R1.2; no longer 3.R3.2
- net D3: now also 4.R1.2; no longer 3.R2.2
- net GND: now also 2.C2.2, 2.C3.2, 2.R4.1, 3.C3.2, 3.R2.1, 3.R3.1, 3.R4.1, 4.C1.2, 4.R3.1, 5.GND1.P$1; no longer 1.C2.2, 2.C0.2, 3.C4.2, 3.C5.2, 3.R5.1, 3.R6.1
- net N$14: now also 2.R3.2; no longer 2.R1.2
- net N$15: now also 2.R4.2; no longer 2.R2.2
- net N$16: now also 3.C4.1; no longer 3.C6.1
- net N$18: now also 3.C4.2; no longer 3.C6.2
- net N$19: now also 2.R2.2; no longer 2.R3.2
- net N$2: now also 2.C3.1; no longer 2.C1.1
- net N$20: now also 3.C5.1; no longer 3.C7.1
- net N$25: now also 3.R3.2; no longer 3.R4.2
- net N$26: now also 3.R4.2; no longer 3.R5.2
- net N$28: now also 3.R2.2; no longer 3.R6.2
- net N$43: now also 4.C1.1, 4.R1.1; no longer 3.C2.1, 3.R2.1
- net N$45: now also 2.C1.1, 2.R1.1; no longer 3.C3.1, 3.R3.1
- net N$5: now also 2.C4.1; no longer 2.C2.1
- net N$6: now also 2.C4.2; no longer 2.C2.2
- net N$8: now also 2.C5.1; no longer 2.C3.1
- net N$9: now also 3.C3.1; no longer 3.C5.1
Other:
- moved on the sheet: 2.C1, 2.C2, 2.C3, 2.R1, 2.R2, 2.R3, 3.C2, 3.C3, 3.C4, 3.C5, 3.R2, 3.R3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
